Commit message: completed implementation and testing of reggie location

File: reggie_support/urdf/reggie.urdf (robot description, URDF)
Before this commit: robot reggie, 5 links, 4 joints
Joints:
- joint chassis_to_left_wheel: origin xyz=0 0.0755 0.0257 rpy=1.5707 0 0 -> xyz=0 0.0755 -0.017 rpy=1.5707 0 0
- joint chassis_to_right_wheel: origin xyz=0 -0.0755 0.0257 rpy=1.5707 0 0 -> xyz=0 -0.0755 -0.017 rpy=1.5707 0 0

Commit message: fixed position of robot model, corrected camera frame id in reggie_support.yaml, removed some obsolete debugging code

File: reggie_support/urdf/reggie.urdf (robot description, URDF)
Before this commit: robot reggie, 5 links, 4 joints
Joints:
- joint base_link_to_chassis: origin xyz=0 0 0 rpy=0 0 0 -> xyz=0 0 0.05 rpy=0 0 0
